File: hss.brd (EAGLE design)
At the start: 41.4 x 29 mm, 11 parts, among them IC1 MEGA328P, Q1 BUZ71

Commit message: Corrected schematic & board
Parts:
- R1, R2: value 3k -> 820
Connections:
- removed net AVCC: IC1.18
- net VCC: now also IC1.18
Routing:
- net VCC: track 76.7 -> 86.1 mm
Changed lines of the file:
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@@
 <?xml version="1.0" encoding="utf-8"?>
 <!DOCTYPE eagle SYSTEM "eagle.dtd">
-<eagle version="6.4">
+<eagle version="6.1">
 <drawing>
 <settings>
@@
 <setting verticaltext="up"/>
 </settings>
-<grid distance="0.01" unitdist="inch" unit="inch" style="lines" multiple="1" display="no" altdistance="0.025" altunitdist="inch" altunit="inch"/>
+<grid distance="0.1" unitdist="inch" unit="inch" style="lines" multiple="1" display="no" altdistance="0.025" altunitdist="inch" altunit="inch"/>
 <layers>
 <layer number="1" name="Top" color="4" fill="1" visible="yes" active="yes"/>
@@
 </class>
 </classes>
-<designrules name="default">
+<designrules>
 <description language="de">&lt;b&gt;EAGLE Design Rules&lt;/b&gt;
 &lt;p&gt;
@@
 <element name="ISP" library="con-lstb" package="MA03-2" value="" x="32.7216625" y="13.909703125" rot="R270"/>
 <element name="C1" library="resistor" package="C1206" value="100nF" x="38.168359375" y="13.793621875" rot="MR90"/>
-<element name="R1" library="resistor" package="M1206" value="3k" x="4.04571875" y="5.92526875" rot="MR0"/>
-<element name="R2" library="resistor" package="M1206" value="3k" x="4.04571875" y="9.123428125" rot="MR0"/>
+<element name="R1" library="resistor" package="M1206" value="820" x="4.04571875" y="5.92526875" rot="MR0"/>
+<element name="R2" library="resistor" package="M1206" value="820" x="4.04571875" y="9.123428125" rot="MR0"/>
 <element name="HITEC" library="con-lstb" package="MA03-1" value="" x="8.56264375" y="6.581853125" rot="R270">
 <attribute name="OC_NEWARK" value="unknown" x="-28.26735625" y="-18.818146875" size="1.778" layer="27" rot="R270" display="off"/>
@@
 <wire x1="8.489490625" y1="12.55938125" x2="4.10708125" y2="12.55938125" width="0.6096" layer="16"/>
 <wire x1="4.10708125" y1="12.55938125" x2="4.10708125" y2="4.032890625" width="0.6096" layer="16"/>
-<wire x1="4.10708125" y1="4.032890625" x2="8.56264375" y2="4.032890625" width="0.6096" layer="16"/>
+<wire x1="4.10708125" y1="4.032890625" x2="8.56264375" y2="4.032890625" width="1.6764" layer="16"/>
 <wire x1="8.56264375" y1="4.032890625" x2="8.56264375" y2="4.041853125" width="0.6096" layer="16"/>
 <wire x1="13.376871875" y1="6.965478125" x2="13.462" y2="6.965478125" width="0.6096" layer="16"/>
 <wire x1="13.462" y1="6.965478125" x2="13.462" y2="7.8704875" width="0.6096" layer="16"/>
-<wire x1="17.01303125" y1="16.726253125" x2="17.80921875" y2="16.736625" width="0" layer="19" extent="16-16"/>
 <wire x1="38.22678125" y1="12.448384375" x2="38.22678125" y2="12.393621875" width="0.6096" layer="16"/>
 <wire x1="38.22678125" y1="12.393621875" x2="38.168359375" y2="12.393621875" width="0.6096" layer="16"/>
+<wire x1="17.80921875" y1="16.736625" x2="17.01303125" y2="16.726253125" width="0" layer="19" extent="16-16"/>
 </signal>
 <signal name="VCC">
@@
 <wire x1="13.17845" y1="19.84435625" x2="17.7778125" y2="19.84435625" width="0.6096" layer="16"/>
 <wire x1="17.7778125" y1="19.84435625" x2="17.81303125" y2="19.807003125" width="0.6096" layer="16"/>
+<contactref element="IC1" pad="18"/>
+<wire x1="20.21303125" y1="9.617103125" x2="20.193" y2="9.617103125" width="0.6096" layer="16"/>
+<wire x1="20.193" y1="9.617103125" x2="20.193" y2="16.129" width="0.6096" layer="16"/>
+<wire x1="20.193" y1="16.129" x2="19.41303125" y2="16.129" width="0.6096" layer="16"/>
+<wire x1="19.41303125" y1="16.129" x2="19.41303125" y2="18.202303125" width="0.6096" layer="16"/>
 <wire x1="34.01130625" y1="16.458890625" x2="33.9916625" y2="16.449703125" width="0" layer="19" extent="16-16"/>
 <wire x1="34.030890625" y1="16.4869625" x2="34.01130625" y2="16.4879125" width="0" layer="19" extent="16-16"/>
-</signal>
-<signal name="AVCC">
-<contactref element="IC1" pad="18"/>
 </signal>
 <signal name="N$1">
@@
 <wire x1="10.705371875" y1="13.539509375" x2="13.782296875" y2="13.539509375" width="0.6096" layer="16"/>
 <wire x1="13.782296875" y1="13.539509375" x2="13.782296875" y2="13.5053125" width="0.6096" layer="16"/>
-<wire x1="8.56264375" y1="9.121853125" x2="8.619903125" y2="9.09396875" width="0" layer="19" extent="16-16"/>
 <wire x1="13.92043125" y1="13.509703125" x2="13.92043125" y2="13.539509375" width="0.6096" layer="16"/>
 <wire x1="13.92043125" y1="13.539509375" x2="13.782296875" y2="13.539509375" width="0.6096" layer="16"/>
+<wire x1="8.619903125" y1="9.09396875" x2="8.56264375" y2="9.121853125" width="0" layer="19" extent="16-16"/>
 </signal>
 <signal name="N$7">
@@
 <signal name="N$6">
 </signal>
-<signal name="N$13">
-<polygon width="0.6096" layer="16" isolate="0.6096" thermals="no">
-<vertex x="0" y="27.94"/>
-<vertex x="40.64" y="27.94"/>
-<vertex x="40.64" y="1.27"/>
-<vertex x="0" y="1.27"/>
-</polygon>
-</signal>
 <signal name="N$15">
 <contactref element="APM" pad="4"/>
@@
 <wire x1="8.5173375" y1="20.20505625" x2="8.5173375" y2="20.20781875" width="0.6096" layer="16"/>
 <contactref element="IC1" pad="30"/>
-<wire x1="8.5173375" y1="20.20505625" x2="8.489490625" y2="20.17938125" width="0" layer="19" extent="16-16"/>
 <wire x1="13.92043125" y1="15.109703125" x2="15.494" y2="15.109703125" width="0.6096" layer="16"/>
 <wire x1="15.494" y1="15.109703125" x2="15.494" y2="16.764" width="0.6096" layer="16"/>
@@
 <wire x1="11.684" y1="19.558" x2="11.684" y2="20.17938125" width="0.6096" layer="16"/>
 <wire x1="11.684" y1="20.17938125" x2="8.489490625" y2="20.17938125" width="0.6096" layer="16"/>
+<wire x1="8.5173375" y1="20.20505625" x2="8.489490625" y2="20.17938125" width="0" layer="19" extent="16-16"/>
 </signal>
 <signal name="N$12">
@@
 <via x="15.494" y="2.286" extent="1-16" drill="0.6" diameter="1.4224"/>
 </signal>
+<signal name="N$13">
+<polygon width="1.27" layer="16" spacing="1.778">
+<vertex x="0" y="0"/>
+<vertex x="0" y="22.86"/>
+<vertex x="40.64" y="22.86"/>
+<vertex x="40.64" y="0"/>
+</polygon>
+</signal>
 </signals>

Commit message: version 4 of the board
Parts:
- removed IN, OUT: MCS08, solpad:MCS08
- removed ISP: (no value), con-lstb:MA03-2
- removed Q1: BUZ71, transistor-fet:TO220
- removed RADIO: (no value), con-lstb:MA04-1
- added C2: 100nF, resistor:C1206
- added LED1: GREEN, led:1206
- added LED2: RED, led:1206
- added R3: 68, resistor:M1206
- added R4: 150, resistor:M1206
- added R5: 10k, resistor:M1206
- APM: device con-lstb:MA04-1 -> con-lstb:MA06-2
- moved C1 17.2 mm to (23.7, 4.52), flipped to the top
- moved R1 15.2 mm to (15.3, 16.2), turned to 180 degrees
- moved R2 11.2 mm to (15.3, 9.42), turned to 180 degrees
- moved HITEC 10.1 mm to (18.3, 4.12), turned to 0 degrees
- moved APM 5.69 mm to (9.65, 10.8), turned to 270 degrees
- moved IC1 2.13 mm to (19.4, 12.1), flipped to the top, turned to 90 degrees
Connections:
- removed net N$11: IN.MP, Q1.3
- net GND: now also APM.2, APM.3, APM.4, LED1.C, LED2.C; no longer ISP.6, RADIO.1
- net N$1: now also IC1.12, R3.1; no longer IC1.29, ISP.5
- net N$10: now also APM.11, APM.12, C2.1; no longer IC1.12, Q1.1
- net N$14: now also APM.10, APM.9; no longer APM.3, RADIO.3
- net N$15: now also APM.7, APM.8; no longer APM.4, RADIO.4
- net N$5: now also C2.2, IC1.29, R5.1; no longer OUT.MP, Q1.2
- net N$7: now also LED1.A, R3.2; no longer IC1.17, ISP.3
- net N$8: now also IC1.13, R4.1; no longer IC1.16, ISP.1
- net N$9: now also LED2.A, R4.2; no longer IC1.15, ISP.4
- net VCC: now also APM.5, APM.6, R5.2; no longer APM.2, ISP.2, RADIO.2
Routing:
- net VCC: track 86.1 -> 44.0 mm, vias 0 -> 2
- net GND: track 75.3 -> 51.6 mm
- net N$1: track 30.7 -> 8.60 mm, vias 4 -> 1
- net N$10: track 26.6 -> 7.86 mm, vias 2 -> 0
- net N$9: track 20.6 -> 4.98 mm, vias 0 -> 1
- net N$3: track 15.3 -> 30.0 mm, vias 0 -> 1
- net N$5: track 2.67 -> 16.3 mm
- net N$7: track 14.8 -> 4.35 mm, vias 0 -> 1
- net N$15: track 16.3 -> 7.28 mm
- net N$8: track 14.3 -> 7.03 mm, vias 0 -> 1
- net N$11: track 4.35 -> 0.00 mm, vias 0 -> 3
- net N$14: track 11.8 -> 8.01 mm
- net N$4: track 13.1 -> 12.6 mm, vias 0 -> 1
- removed copper zone on layer 16, net N$13
Other:
- board size 41.4 x 29 mm -> 27.7 x 17.6 mm
- board text added: "APM-HSS"
- board text added: "Adapter"
- board text added: "Janne Mäntyharju"
- board text added: "Rev 4"
